File: car.sch (KiCad schematic (older format))
At the start: 3 parts, among them J1 Subaru_ECM, J2 Conn_02x20_Counter_Clockwise

Commit message: Rework wiring
- Add auxiliary connector
- Add switches to auxiliar6 connector
- Add COP wiring to auxiliary connector
- Rework ground plane
Parts:
- added J?: Aptiv_Micropak100_24p, symbol Connector_Aptiv:Aptiv_Micropak100_24p
- J1: symbol MCU_Microchip_PIC16:Subaru_ECM -> car-rescue:Subaru_ECM-MCU_Microchip_PIC16
Connections:
- net labels added: +12v_Screw_Terminal, Aux_Idle_Stepper_1A, Aux_Idle_Stepper_1B, Aux_Idle_Stepper_2A, Aux_Idle_Stepper_2B, Aux_Ignition_1, Aux_Ignition_2, Aux_Ignition_3, Aux_Ignition_4, Aux_VVT1, Aux_VVT2, Fan_Override_Switch, Fuel_Pmp_SW, Ground_G1, Ground_G2, Ground_Shield_Joint, Ground_VR_Shield, Ignition_Switched_Power
- net labels removed: Idle_Stepper_1A, Idle_Stepper_1B, Idle_Stepper_2A, Idle_Stepper_2B, Ignition_3, Ignition_4, PWM_Idle, Proto_3B, VVT
- wire segments 67 -> 96
Other:
- moved on the sheet: MH1
Changed lines of the file:
@@
 EESchema Schematic File Version 4
-EELAYER 26 0
+LIBS:car-cache
+EELAYER 29 0
 EELAYER END
 $Descr USLetter 11000 8500
@@
 Comment4 ""
 $EndDescr
-$Comp
-L MCU_Microchip_PIC16:Subaru_ECM J1
-U 1 1 5BB1DA41
-P 2050 2500
-F 0 "J1" H 1300 2600 50  0000 R CNN
-F 1 "Subaru_ECM" H 1550 2800 50  0000 R CNN
-F 2 "Connector:Subaru ECM Connector" H 2050 2350 50  0001 C CNN
-F 3 "" H 2050 2350 50  0001 C CNN
-	1    2050 2500
-	1    0    0    -1
-$EndComp
 Text Label 7950 1800 2    50   ~ 0
 Injector_1_1
@@
 Injector_4_2
 Text Label 7950 2400 2    50   ~ 0
-Ignition_1
+Aux_Ignition_1
 Text Label 7950 2500 2    50   ~ 0
-Ignition_4
+Aux_Ignition_4
 Text Label 7950 2600 2    50   ~ 0
-Ground
+Ground_G1
 Text Label 7950 2700 2    50   ~ 0
-Ground
+Ground_G2
 Text Label 7950 2800 2    50   ~ 0
 MAP_0-5v
 Text Label 7950 2900 2    50   ~ 0
-Ground
+Ground_VR_Shield
 Text Label 7950 3000 2    50   ~ 0
 5v
@@
 TPS_Input
 Text Label 9200 3500 0    50   ~ 0
-Ground
+Ground_Shield_Joint
 Text Label 9200 3400 0    50   ~ 0
 Cam_Input_VR2+
@@
 5v
 Text Label 9200 2900 0    50   ~ 0
-Idle_Stepper_2B
+Aux_Idle_Stepper_2B
 Text Label 9200 2800 0    50   ~ 0
-Idle_Stepper_2A
+Aux_Idle_Stepper_2A
 Text Label 9200 2700 0    50   ~ 0
-Idle_Stepper_1A
+Aux_Idle_Stepper_1A
 Text Label 9200 2600 0    50   ~ 0
-Idle_Stepper_1B
+Aux_Idle_Stepper_1B
 Text Label 9200 2500 0    50   ~ 0
-Ignition_3
+Aux_Ignition_3
 Text Label 9200 2400 0    50   ~ 0
-Ignition_2
+Aux_Ignition_2
 Text Label 9200 2300 0    50   ~ 0
 Boost
@@
 Idle_2
 Text Label 9200 2100 0    50   ~ 0
-PWM_Idle
+Aux_VVT2
 Text Label 9200 2000 0    50   ~ 0
-VVT
+Aux_VVT1
 Text Label 9200 1900 0    50   ~ 0
 Injector_2_2?
@@
 Text Label 1400 5500 2    50   ~ 0
 Injector_4_1
-Text Label 4800 1100 1    50   ~ 0
-Ignition_1
 Text Label 3200 1100 1    50   ~ 0
 MAP_0-5v
 Text Label 3900 1100 1    50   ~ 0
-Proto_3B
+Fuel_Pmp_SW
 Text Label 2800 1100 1    50   ~ 0
 Coolant
 Text Label 1400 3400 2    50   ~ 0
 Intake_Air_Temp
-Text Label 4700 1100 1    50   ~ 0
-Ignition_2
 Text Label 3500 1100 1    50   ~ 0
 VR1-
@@
 	1400 5500 1600 5500
 Wire Wire Line
-	5000 6800 5000 6550
-Wire Wire Line
-	5850 5400 6100 5400
-Wire Wire Line
 	5100 1100 5100 1350
 Wire Wire Line
@@
 L power:GND #PWR0101
 U 1 1 5BB3C560
-P 7600 5450
-F 0 "#PWR0101" H 7600 5200 50  0001 C CNN
-F 1 "GND" H 7605 5277 50  0000 C CNN
-F 2 "" H 7600 5450 50  0001 C CNN
-F 3 "" H 7600 5450 50  0001 C CNN
-	1    7600 5450
+P 8500 1150
+F 0 "#PWR0101" H 8500 900 50  0001 C CNN
+F 1 "GND" H 8505 977 50  0000 C CNN
+F 2 "" H 8500 1150 50  0001 C CNN
+F 3 "" H 8500 1150 50  0001 C CNN
+	1    8500 1150
 	1    0    0    -1
 $EndComp
-Text Label 7750 5450 0    50   ~ 0
+Text Label 8650 1150 0    50   ~ 0
 Ground
 Text Label 6100 5300 0    50   ~ 0
-Ground
+Ground_G1
 Text Label 6100 2900 0    50   ~ 0
-Ground
+Ground_G1
 Text Label 4900 1100 1    50   ~ 0
-Ground
+Ground_G1
 Text Label 2500 1100 1    50   ~ 0
-Ground
+Ground_G1
 Text Label 2400 1100 1    50   ~ 0
+Ground_G2
+Text Label 2300 1100 1    50   ~ 0
+Ground_G2
+Text Label 3400 6800 3    50   ~ 0
+Ground_G2
+Text Label 4900 6800 3    50   ~ 0
+Ground_G2
+Text Label 8350 1150 2    50   ~ 0
 NPS_Ground
-Text Label 2300 1100 1    50   ~ 0
-NPS_Ground
-Text Label 3400 6800 3    50   ~ 0
-NPS_Ground
-Text Label 4900 6800 3    50   ~ 0
-Ground
-Text Label 7450 5450 2    50   ~ 0
-NPS_Ground
-Wire Wire Line
-	5850 5300 6100 5300
-Wire Wire Line
-	5850 2900 6100 2900
 Wire Wire Line
 	4900 1100 4900 1350
@@
 Wire Wire Line
 	2500 1100 2500 1350
-Wire Wire Line
-	3400 6800 3400 6550
-Wire Wire Line
-	4900 6800 4900 6550
 $Comp
 L Mechanical:MountingHole_Pad MH1
 U 1 1 5BB4A7DE
-P 7600 5150
-F 0 "MH1" H 7700 5201 50  0000 L CNN
-F 1 "MountingHole_Pad" H 7700 5110 50  0000 L CNN
-F 2 "MountingHole:MountingHole_3.5mm_Pad" H 7600 5150 50  0001 C CNN
-F 3 "~" H 7600 5150 50  0001 C CNN
-	1    7600 5150
+P 8500 850
+F 0 "MH1" H 8600 901 50  0000 L CNN
+F 1 "MountingHole_Pad" H 8600 810 50  0000 L CNN
+F 2 "MountingHole:MountingHole_3.5mm_Pad" H 8500 850 50  0001 C CNN
+F 3 "~" H 8500 850 50  0001 C CNN
+	1    8500 850
 	1    0    0    -1
 $EndComp
 Wire Wire Line
-	7600 5250 7600 5450
-Wire Wire Line
-	7450 5450 7600 5450
-Connection ~ 7600 5450
-Wire Wire Line
-	7750 5450 7600 5450
+	8500 950  8500 1150
+Wire Wire Line
+	8350 1150 8500 1150
+Connection ~ 8500 1150
+Wire Wire Line
+	8650 1150 8500 1150
 $Comp
 L Connector_Generic:Conn_02x20_Counter_Clockwise J2
@@
 Wire Wire Line
 	2700 1100 2700 1350
+Wire Wire Line
+	5850 5400 6100 5400
+Wire Wire Line
+	5850 5300 6100 5300
+Wire Wire Line
+	5850 2900 6100 2900
+Wire Wire Line
+	5000 6800 5000 6550
+Wire Wire Line
+	4900 6800 4900 6550
+Wire Wire Line
+	3400 6800 3400 6550
+Text Label 6100 4800 0    50   ~ 0
+Proto_4A
+$Comp
+L car-rescue:Subaru_ECM-MCU_Microchip_PIC16 J1
+U 1 1 5BB1DA41
+P 2050 2500
+F 0 "J1" H 1300 2600 50  0000 R CNN
+F 1 "Subaru_ECM" H 1550 2800 50  0000 R CNN
+F 2 "Connector:Subaru ECM Connector" H 2050 2350 50  0001 C CNN
+F 3 "" H 2050 2350 50  0001 C CNN
+	1    2050 2500
+	1    0    0    -1
+$EndComp
+Text Label 2900 1100 1    50   ~ 0
+O2_Sensor
+Wire Wire Line
+	2900 1100 2900 1350
+Text Label 1400 2700 2    50   ~ 0
++12v_Screw_Terminal
+Wire Wire Line
+	1400 2700 1600 2700
+Text Label 1400 2800 2    50   ~ 0
++12v_Screw_Terminal
+Wire Wire Line
+	1400 2800 1600 2800
+Text Label 4800 1100 1    50   ~ 0
+Ignition_1
+Text Label 4700 1100 1    50   ~ 0
+Ignition_2
+Text Label 2600 6800 3    50   ~ 0
+Fan_Override_Switch
+Wire Wire Line
+	2600 6800 2600 6550
+Wire Wire Line
+	2700 6800 2700 6550
+Text Label 2500 6800 3    50   ~ 0
+Proto_5A
+Wire Wire Line
+	2500 6800 2500 6550
+Text Label 2600 1100 1    50   ~ 0
+Ground_Shield_Joint
+Wire Wire Line
+	2600 1100 2600 1350
+Text Label 6100 4000 0    50   ~ 0
+Ground_Shield_Joint
+Text Label 6100 3900 0    50   ~ 0
+Ground_Shield_Joint
+Wire Wire Line
+	6100 3900 5850 3900
+Wire Wire Line
+	5850 4000 6100 4000
+Text Label 6100 3700 0    50   ~ 0
+Ground_VR_Shield
+Wire Wire Line
+	6100 3700 5850 3700
+Text Label 4500 1100 1    50   ~ 0
+Ground_Shield_Joint
+Wire Wire Line
+	4500 1100 4500 1350
+Text Label 4800 6800 3    50   ~ 0
+Ground_G2
+Wire Wire Line
+	4800 6800 4800 6550
+$Comp
+L Connector_Aptiv:Aptiv_Micropak100_24p J?
+U 1 1 5CF96E65
+P 8500 4950
+F 0 "J?" H 8550 5667 50  0000 C CNN
+F 1 "Aptiv_Micropak100_24p" H 8550 5576 50  0000 C CNN
+F 2 "" H 8500 4950 50  0001 C CNN
+F 3 "~" H 8500 4950 50  0001 C CNN
+	1    8500 4950
+	1    0    0    -1
+$EndComp
+Text Label 7600 4550 0    50   ~ 0
+Aux_Ignition_2
+Text Label 7600 4450 0    50   ~ 0
+Aux_Ignition_1
+Text Label 7600 4650 0    50   ~ 0
+Aux_Ignition_3
+Text Label 7600 4750 0    50   ~ 0
+Aux_Ignition_4
+Wire Wire Line
+	8150 4450 8300 4450
+Wire Wire Line
+	8150 4550 8300 4550
+Wire Wire Line
+	8150 4650 8300 4650
+Wire Wire Line
+	8150 4750 8300 4750
+Text Label 7800 4850 0    50   ~ 0
+Aux_VVT1
+Wire Wire Line
+	8150 4850 8300 4850
+Wire Wire Line
+	8150 4950 8300 4950
+Text Label 7800 4950 0    50   ~ 0
+Aux_VVT2
+Wire Wire Line
+	8150 5050 8300 5050
+Wire Wire Line
+	8150 5150 8300 5150
+Text Label 7650 5050 0    50   ~ 0
+Fuel_Pmp_SW
+Text Label 7800 5150 0    50   ~ 0
+Proto_3A
+Text Label 3900 6800 3    50   ~ 0
+Ignition_Switched_Power
+Wire Wire Line
+	3900 6800 3900 6550
+Text Label 6100 4700 0    50   ~ 0
+Ignition_Switched_Power
+Wire Wire Line
+	5850 4800 6100 4800
+Wire Wire Line
+	6100 4700 5850 4700
+Text Label 7250 5250 0    50   ~ 0
+Ignition_Switched_Power
+Wire Wire Line
+	8150 5250 8300 5250
+Text Label 8150 5350 2    50   ~ 0
+Proto_2A
+Wire Wire Line
+	8150 5350 8300 5350
+Text Label 2700 6800 3    50   ~ 0
+Fan_Override_Switch
+Text Label 9200 4750 0    50   ~ 0
+Aux_Idle_Stepper_2B
+Text Label 9200 4650 0    50   ~ 0
+Aux_Idle_Stepper_2A
+Text Label 9200 4550 0    50   ~ 0
+Aux_Idle_Stepper_1A
+Text Label 9200 4450 0    50   ~ 0
+Aux_Idle_Stepper_1B
+Wire Wire Line
+	9200 4450 8800 4450
+Wire Wire Line
+	8800 4550 9200 4550
+Wire Wire Line
+	9200 4650 8800 4650
+Wire Wire Line
+	8800 4750 9200 4750
 $EndSCHEMATC
